File: hardware/mainBoard/mainBoard.kicad_sch (KiCad schematic)
At the start: 19 parts, among them J1 UARTDebug, J2 LeftKeyConnector, J3 DisplayConnector, J4 RightKeyConnector, J5 EncoderConnector, U1 MCP4728-E_UN

Commit message: update wrong ldac pin
Connections:
- net LDAC: now also A1.17 (GPIO13); no longer A1.20 (GPIO15)
- no-connect marks 11 -> 10
Changed lines of the file:
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@@
 		(at 64.77 78.74)
 	)
-	(no_connect
-		(at 64.77 81.28)
-	)
 	(wire
 		(pts
@@
 	)
 	(label "LDAC"
-		(at 64.77 86.36 180)
+		(at 64.77 81.28 180)
 		(effects
 			(font
