File: hardware/mainBoard/mainBoard.kicad_pcb (KiCad board)
At the start: 2 copper layers, 99.9 x 52.5 mm, 24 parts, among them J1 UARTDebug, J2 LeftKeyConnector, J3 DisplayConnector, J4 LEDHeader, J5 RightKeyConnector, J6 EncoderConnector, U1 MCP4728-E_UN

Commit message: update resistor size
Parts:
- R1, R2, R3, R4: value 680 -> 665
Changed lines of the file:
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@@
 			)
 		)
-		(property "Value" "680"
+		(property "Value" "665"
 			(at 0 1.83 0)
 			(layer "F.Fab")
@@
 			)
 		)
-		(property "LCSC Part #" "C137240"
+		(property "LCSC Part #" "C54532953"
 			(at 0 0 180)
 			(unlocked yes)
@@
 			)
 		)
-		(property "Price" " $0.0066 "
+		(property "Price" " $0.0059 "
 			(at 0 0 180)
 			(unlocked yes)
@@
 			)
 		)
-		(property "Value" "680"
+		(property "Value" "665"
 			(at 0 1.83 0)
 			(layer "F.Fab")
@@
 			)
 		)
-		(property "LCSC Part #" "C137240"
+		(property "LCSC Part #" "C54532953"
 			(at 0 0 180)
 			(unlocked yes)
@@
 			)
 		)
-		(property "Price" " $0.0066 "
+		(property "Price" " $0.0059 "
 			(at 0 0 180)
 			(unlocked yes)
@@
 			)
 		)
-		(property "Value" "680"
+		(property "Value" "665"
 			(at 0 1.83 0)
 			(layer "F.Fab")
@@
 			)
 		)
-		(property "LCSC Part #" "C137240"
+		(property "LCSC Part #" "C54532953"
 			(at 0 0 180)
 			(unlocked yes)
@@
 			)
 		)
-		(property "Price" " $0.0066 "
+		(property "Price" " $0.0059 "
 			(at 0 0 180)
 			(unlocked yes)
@@
 			)
 		)
-		(property "Value" "680"
+		(property "Value" "665"
 			(at 0 1.83 0)
 			(layer "F.Fab")
@@
 			)
 		)
-		(property "LCSC Part #" "C137240"
+		(property "LCSC Part #" "C54532953"
 			(at 0 0 180)
 			(unlocked yes)
@@
 			)
 		)
-		(property "Price" " $0.0066 "
+		(property "Price" " $0.0059 "
 			(at 0 0 180)
 			(unlocked yes)
