File: hardware/inputBoard/inputBoard.kicad_sch (KiCad schematic)
At the start: 12 parts, among them J2 LeftKeyConnector, J3 RightKeyConnector, J4 EncoderConnector, SW1 SW_Push, SW2 SW_Push, SW3 SW_Push, SW4 SW_Push, SW5 SW_Push, SW6 SW_Push, SW7 SW_Push, SW8 SW_Push, SW9 RotaryEncoder_Switch_MP

Commit message: Label the connectors in the silkscreen
Changed lines of the file:
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@@
+	(wire
+		(pts
+			(xy 43.18 124.46) (xy 43.18 118.11)
+		)
+		(stroke
+			(width 0)
+			(type default)
+		)
+	)
 	(wire
 		(pts
@@
 				)
 			)
-			(project "anadashSecondaryBoard"
+			(project "inputBoard"
 				(path "/4afd32ea-561a-4b0e-b8bd-b5545b1531de"
 					(reference "SW9")
@@
 				)
 			)
-			(project "anadashSecondaryBoard"
+			(project "inputBoard"
 				(path "/4afd32ea-561a-4b0e-b8bd-b5545b1531de"
 					(reference "SW5")
@@
 				)
 			)
-			(project "anadashSecondaryBoard"
+			(project "inputBoard"
 				(path "/4afd32ea-561a-4b0e-b8bd-b5545b1531de"
 					(reference "SW7")
@@
 				)
 			)
-			(project "anadashSecondaryBoard"
+			(project "inputBoard"
 				(path "/4afd32ea-561a-4b0e-b8bd-b5545b1531de"
 					(reference "SW8")
@@
 				)
 			)
-			(project "anadashSecondaryBoard"
+			(project "inputBoard"
 				(path "/4afd32ea-561a-4b0e-b8bd-b5545b1531de"
 					(reference "J4")
@@
 				)
 			)
-			(project "anadashSecondaryBoard"
+			(project "inputBoard"
 				(path "/4afd32ea-561a-4b0e-b8bd-b5545b1531de"
 					(reference "#PWR06")
@@
 				)
 			)
-			(project "anadashSecondaryBoard"
+			(project "inputBoard"
 				(path "/4afd32ea-561a-4b0e-b8bd-b5545b1531de"
 					(reference "SW4")
@@
 				)
 			)
-			(project "anadashSecondaryBoard"
+			(project "inputBoard"
 				(path "/4afd32ea-561a-4b0e-b8bd-b5545b1531de"
 					(reference "SW3")
@@
 				)
 			)
-			(project "anadashSecondaryBoard"
+			(project "inputBoard"
 				(path "/4afd32ea-561a-4b0e-b8bd-b5545b1531de"
 					(reference "SW6")
@@
 				)
 			)
-			(project "anadashSecondaryBoard"
+			(project "inputBoard"
 				(path "/4afd32ea-561a-4b0e-b8bd-b5545b1531de"
 					(reference "J2")
@@
 		)
 		(instances
-			(project "anadashSecondaryBoard"
+			(project "inputBoard"
 				(path "/4afd32ea-561a-4b0e-b8bd-b5545b1531de"
 					(reference "#PWR03")
@@
 		)
 		(instances
-			(project "anadashSecondaryBoard"
+			(project "inputBoard"
 				(path "/4afd32ea-561a-4b0e-b8bd-b5545b1531de"
 					(reference "#PWR02")
@@
 				)
 			)
-			(project "anadashSecondaryBoard"
+			(project "inputBoard"
 				(path "/4afd32ea-561a-4b0e-b8bd-b5545b1531de"
 					(reference "SW1")
@@
 	(symbol
 		(lib_id "power:GND")
-		(at 43.18 118.11 0)
+		(at 43.18 124.46 0)
 		(unit 1)
 		(body_style 1)
@@
 		(fields_autoplaced yes)
 		(property "Reference" "#PWR01"
+			(at 43.18 130.81 0)
+			(hide yes)
+			(show_name no)
+			(do_not_autoplace no)
+			(effects
+				(font
+					(size 1.27 1.27)
+				)
+			)
+		)
+		(property "Value" "GND"
+			(at 43.18 129.54 0)
+			(show_name no)
+			(do_not_autoplace no)
+			(effects
+				(font
+					(size 1.27 1.27)
+				)
+			)
+		)
+		(property "Footprint" ""
 			(at 43.18 124.46 0)
 			(hide yes)
@@
 			)
 		)
-		(property "Value" "GND"
-			(at 43.18 123.19 0)
-			(show_name no)
-			(do_not_autoplace no)
-			(effects
-				(font
-					(size 1.27 1.27)
-				)
-			)
-		)
-		(property "Footprint" ""
-			(at 43.18 118.11 0)
-			(hide yes)
-			(show_name no)
-			(do_not_autoplace no)
-			(effects
-				(font
-					(size 1.27 1.27)
-				)
-			)
-		)
 		(property "Datasheet" ""
-			(at 43.18 118.11 0)
+			(at 43.18 124.46 0)
 			(hide yes)
 			(show_name no)
@@
 		)
 		(property "Description" "Power symbol creates a global label with name \"GND\" , ground"
-			(at 43.18 118.11 0)
+			(at 43.18 124.46 0)
 			(hide yes)
 			(show_name no)
@@
 		)
 		(instances
-			(project "anadashSecondaryBoard"
+			(project "inputBoard"
 				(path "/4afd32ea-561a-4b0e-b8bd-b5545b1531de"
 					(reference "#PWR01")
@@
 				)
 			)
-			(project "anadashSecondaryBoard"
+			(project "inputBoard"
 				(path "/4afd32ea-561a-4b0e-b8bd-b5545b1531de"
 					(reference "SW2")
@@
 				)
 			)
-			(project "anadashSecondaryBoard"
+			(project "inputBoard"
 				(path "/4afd32ea-561a-4b0e-b8bd-b5545b1531de"
 					(reference "J3")

Commit message: update PCB routing and add debug probe
Parts:
- renumbered J2 to J101, J3 to J102, J4 to J103, SW1 to SW101, SW2 to SW102, SW3 to SW103, SW4 to SW104, SW5 to SW105, SW6 to SW106, SW7 to SW107, SW8 to SW108, SW9 to SW109
Changed lines of the file:
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@@
 		(dnp no)
 		(fields_autoplaced yes)
-		(property "Reference" "SW9"
+		(property "Reference" "SW109"
 			(at 59.69 151.13 0)
 			(show_name no)
@@
 			(project "inputBoard"
 				(path "/4afd32ea-561a-4b0e-b8bd-b5545b1531de"
-					(reference "SW9")
+					(reference "SW109")
 					(unit 1)
 				)
@@
 		(dnp no)
 		(fields_autoplaced yes)
-		(property "Reference" "SW5"
+		(property "Reference" "SW105"
 			(at 59.69 100.33 0)
 			(show_name no)
@@
 			(project "inputBoard"
 				(path "/4afd32ea-561a-4b0e-b8bd-b5545b1531de"
-					(reference "SW5")
+					(reference "SW105")
 					(unit 1)
 				)
@@
 		(dnp no)
 		(fields_autoplaced yes)
-		(property "Reference" "SW7"
+		(property "Reference" "SW107"
 			(at 59.69 120.65 0)
 			(show_name no)
@@
 			(project "inputBoard"
 				(path "/4afd32ea-561a-4b0e-b8bd-b5545b1531de"
-					(reference "SW7")
+					(reference "SW107")
 					(unit 1)
 				)
@@
 		(dnp no)
 		(fields_autoplaced yes)
-		(property "Reference" "SW8"
+		(property "Reference" "SW108"
 			(at 59.69 130.81 0)
 			(show_name no)
@@
 			(project "inputBoard"
 				(path "/4afd32ea-561a-4b0e-b8bd-b5545b1531de"
-					(reference "SW8")
+					(reference "SW108")
 					(unit 1)
 				)
@@
 		(in_pos_files yes)
 		(dnp no)
-		(property "Reference" "J4"
+		(property "Reference" "J103"
 			(at 55.88 182.88 90)
 			(show_name no)
@@
 			(project "inputBoard"
 				(path "/4afd32ea-561a-4b0e-b8bd-b5545b1531de"
-					(reference "J4")
+					(reference "J103")
 					(unit 1)
 				)
@@
 		(dnp no)
 		(fields_autoplaced yes)
-		(property "Reference" "#PWR06"
+		(property "Reference" "#PWR0103"
 			(at 68.58 109.22 0)
 			(hide yes)
@@
 			(project "inputBoard"
 				(path "/4afd32ea-561a-4b0e-b8bd-b5545b1531de"
-					(reference "#PWR06")
+					(reference "#PWR0103")
 					(unit 1)
 				)
@@
 		(dnp no)
 		(fields_autoplaced yes)
-		(property "Reference" "SW4"
+		(property "Reference" "SW104"
 			(at 59.69 90.17 0)
 			(show_name no)
@@
 			(project "inputBoard"
 				(path "/4afd32ea-561a-4b0e-b8bd-b5545b1531de"
-					(reference "SW4")
+					(reference "SW104")
 					(unit 1)
 				)
@@
 		(dnp no)
 		(fields_autoplaced yes)
-		(property "Reference" "SW3"
+		(property "Reference" "SW103"
 			(at 59.69 80.01 0)
 			(show_name no)
@@
 			(project "inputBoard"
 				(path "/4afd32ea-561a-4b0e-b8bd-b5545b1531de"
-					(reference "SW3")
+					(reference "SW103")
 					(unit 1)
 				)
@@
 		(dnp no)
 		(fields_autoplaced yes)
-		(property "Reference" "SW6"
+		(property "Reference" "SW106"
 			(at 59.69 110.49 0)
 			(show_name no)
@@
 			(project "inputBoard"
 				(path "/4afd32ea-561a-4b0e-b8bd-b5545b1531de"
-					(reference "SW6")
+					(reference "SW106")
 					(unit 1)
 				)
@@
 		(in_pos_files yes)
 		(dnp no)
-		(property "Reference" "J2"
+		(property "Reference" "J101"
 			(at 38.1 104.14 0)
 			(show_name no)
@@
 			(project "inputBoard"
 				(path "/4afd32ea-561a-4b0e-b8bd-b5545b1531de"
-					(reference "J2")
+					(reference "J101")
 					(unit 1)
 				)
@@
 		(dnp no)
 		(fields_autoplaced yes)
-		(property "Reference" "#PWR03"
+		(property "Reference" "#PWR0104"
 			(at 69.85 176.53 0)
 			(hide yes)
@@
 			(project "inputBoard"
 				(path "/4afd32ea-561a-4b0e-b8bd-b5545b1531de"
-					(reference "#PWR03")
+					(reference "#PWR0104")
 					(unit 1)
 				)
@@
 		(dnp no)
 		(fields_autoplaced yes)
-		(property "Reference" "#PWR02"
+		(property "Reference" "#PWR0102"
 			(at 50.8 104.14 0)
 			(hide yes)
@@
 			(project "inputBoard"
 				(path "/4afd32ea-561a-4b0e-b8bd-b5545b1531de"
-					(reference "#PWR02")
+					(reference "#PWR0102")
 					(unit 1)
 				)
@@
 		(dnp no)
 		(fields_autoplaced yes)
-		(property "Reference" "SW1"
+		(property "Reference" "SW101"
 			(at 59.69 59.69 0)
 			(show_name no)
@@
 			(project "inputBoard"
 				(path "/4afd32ea-561a-4b0e-b8bd-b5545b1531de"
-					(reference "SW1")
+					(reference "SW101")
 					(unit 1)
 				)
@@
 		(dnp no)
 		(fields_autoplaced yes)
-		(property "Reference" "#PWR01"
+		(property "Reference" "#PWR0101"
 			(at 43.18 130.81 0)
 			(hide yes)
@@
 			(project "inputBoard"
 				(path "/4afd32ea-561a-4b0e-b8bd-b5545b1531de"
-					(reference "#PWR01")
+					(reference "#PWR0101")
 					(unit 1)
 				)
@@
 		(dnp no)
 		(fields_autoplaced yes)
-		(property "Reference" "SW2"
+		(property "Reference" "SW102"
 			(at 59.69 69.85 0)
 			(show_name no)
@@
 			(project "inputBoard"
 				(path "/4afd32ea-561a-4b0e-b8bd-b5545b1531de"
-					(reference "SW2")
+					(reference "SW102")
 					(unit 1)
 				)
@@
 		(in_pos_files yes)
 		(dnp no)
-		(property "Reference" "J3"
+		(property "Reference" "J102"
 			(at 38.1 124.46 0)
 			(show_name no)
@@
 			(project "inputBoard"
 				(path "/4afd32ea-561a-4b0e-b8bd-b5545b1531de"
-					(reference "J3")
-					(unit 1)
-				)
+					(reference "J102")
+					(unit 1)
+				)

Commit message: add production files
Parts:
- J101, J102: LCSC Part # (none) -> C157991; Price (none) -> $0.0878
- J103: LCSC Part # (none) -> C144395; Price (none) -> $0.0574
- SW101, SW102, SW103, SW104, SW105, SW106, SW107, SW108: LCSC Part # (none) -> N/A; Price (none) -> $0.265
- SW109: LCSC Part # (none) -> C370986; Price (none) -> $2.2797

Commit message: update production files + start miscellaneous bom
Parts:
- J101, J102: LCSC Price (none) -> $0.0878; Price $0.0878 -> (none)
- J103: LCSC Price (none) -> $0.0574; Price $0.0574 -> (none)
- SW101, SW102, SW103, SW104, SW105, SW106, SW107, SW108: AliExpress Link (none) -> https://pt.aliexpress.com/item/1005010462521108.html; AliExpress Price (none) -> $0,0265; LCSC Price (none) -> N/A; Price $0.265 -> (none)
- SW109: LCSC Price (none) -> $2.2797; Price $2.2797 -> (none)
