File: hardware/inputBoard/inputBoard.kicad_pcb (KiCad board)
At the start: 2 copper layers, 198 x 34 mm, 17 parts, among them J101 LeftKeyConnector, J102 RightKeyConnector, J103 EncoderConnector, SW101 SW_Push, SW102 SW_Push, SW103 SW_Push, SW104 SW_Push, SW105 SW_Push, SW106 SW_Push, SW107 SW_Push, SW108 SW_Push, SW109 RotaryEncoder_Switch_MP

Commit message: update inputboard to use one layer only
Routing:
- net Net-(J103-Pin_3): track 23.2 -> 22.1 mm
Changed lines of the file:
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@@
 		(tags "rotary encoder")
 		(property "Reference" "SW109"
-			(at 2.8 -4.7 0)
+			(at 7.25 -5.819125 0)
 			(layer "F.SilkS")
 			(effects
@@
 	)
 	(segment
-		(start 152.79 94.979125)
-		(end 154.671428 94.979125)
+		(start 157.34 76.279125)
+		(end 157.34 90.429125)
 		(width 0.2)
-		(layer "B.Cu")
-		(net "Net-(J103-Pin_3)")
-	)
-	(segment
-		(start 155.671428 93.979125)
-		(end 155.671428 85.579125)
-		(width 0.2)
-		(layer "B.Cu")
-		(net "Net-(J103-Pin_3)")
-	)
-	(segment
-		(start 155.671428 85.579125)
-		(end 157.34 83.910553)
-		(width 0.2)
-		(layer "B.Cu")
-		(net "Net-(J103-Pin_3)")
-	)
-	(segment
-		(start 157.34 83.910553)
-		(end 157.34 76.279125)
-		(width 0.2)
-		(layer "B.Cu")
-		(net "Net-(J103-Pin_3)")
-	)
-	(segment
-		(start 154.671428 94.979125)
-		(end 155.671428 93.979125)
-		(width 0.2)
-		(layer "B.Cu")
+		(layer "F.Cu")
 		(net "Net-(J103-Pin_3)")
 	)
 	(segment
-		(start 151.75 96.019125)
-		(end 152.79 94.979125)
+		(start 157.34 90.429125)
+		(end 151.75 96.019125)
 		(width 0.2)
-		(layer "B.Cu")
+		(layer "F.Cu")
 		(net "Net-(J103-Pin_3)")
 	)
