File: hardware/inputBoard/inputBoard.kicad_pcb (KiCad board)
At the start: 2 copper layers, 198 x 34 mm, 17 parts, among them J101 LeftKeyConnector, J102 RightKeyConnector, J103 EncoderConnector, SW101 SW_Push, SW102 SW_Push, SW103 SW_Push, SW104 SW_Push, SW105 SW_Push, SW106 SW_Push, SW107 SW_Push, SW108 SW_Push, SW109 RotaryEncoder_Switch_MP

Commit message: update inputboard
Parts:
- moved G*** 56.2 mm to (144.2, 77.0)
- moved REF** 16.7 mm to (82.7, 77.0)
- moved REF** 16.7 mm to (235.3, 77.0)
- moved SW101 11.4 mm to (85.2, 88.4)
- moved SW108 11.4 mm to (237.9, 88.4)
- moved SW107 9.19 mm to (218.6, 88.4)
- moved SW102 9.16 mm to (104.5, 88.4)
- moved SW103 6.91 mm to (123.7, 88.4)
- moved SW106 6.91 mm to (199.4, 88.4)
- moved SW105 4.68 mm to (180.1, 88.4)
- moved SW104 4.66 mm to (143.0, 88.4)
Routing:
- net Net-(J102-Pin_2): track 31.8 -> 20.4 mm
- net Net-(J101-Pin_5): track 33.0 -> 21.6 mm
- net GND: track 0.00 -> 9.07 mm
- net Net-(J102-Pin_4): track 16.8 -> 23.2 mm
- net Net-(J101-Pin_3): track 16.3 -> 22.0 mm
- net Net-(J102-Pin_5): track 35.3 -> 40.0 mm
- net Net-(J101-Pin_2): track 34.1 -> 38.8 mm
- net Net-(J101-Pin_4): track 15.9 -> 12.3 mm
- net Net-(J102-Pin_3): track 15.4 -> 12.8 mm
Other:
- board size 198 x 34 mm -> 173 x 34 mm
- board text added: "AnaDash InputBoard"
Changed lines of the file:
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@@
 	(footprint "Designs:tinycat"
 		(layer "F.Cu")
-		(at 88 77)
+		(at 144.25 77)
 		(property "Reference" "G***"
 			(at 0 0 0)
@@
 	(footprint "footprints:SW_Cherry_MX_1.00u_PCB"
 		(layer "F.Cu")
-		(at 138.305 88.439125)
+		(at 142.96 88.439125)
 		(descr "Cherry MX keyswitch, 1.00u, PCB mount, http://cherryamericas.com/wp-content/uploads/2014/12/mx_cat.pdf")
 		(tags "Cherry MX keyswitch 1.00u PCB")
@@
 	(footprint "footprints:SW_Cherry_MX_1.00u_PCB"
 		(layer "F.Cu")
-		(at 95.295 88.439125)
+		(at 104.46 88.439125)
 		(descr "Cherry MX keyswitch, 1.00u, PCB mount, http://cherryamericas.com/wp-content/uploads/2014/12/mx_cat.pdf")
 		(tags "Cherry MX keyswitch 1.00u PCB")
@@
 	(footprint "footprints:SW_Cherry_MX_1.00u_PCB"
 		(layer "F.Cu")
-		(at 206.28 88.439125)
+		(at 199.37 88.439125)
 		(descr "Cherry MX keyswitch, 1.00u, PCB mount, http://cherryamericas.com/wp-content/uploads/2014/12/mx_cat.pdf")
 		(tags "Cherry MX keyswitch 1.00u PCB")
@@
 	(footprint "footprints:SW_Cherry_MX_1.00u_PCB"
 		(layer "F.Cu")
-		(at 184.775 88.439125)
+		(at 180.1 88.439125)
 		(descr "Cherry MX keyswitch, 1.00u, PCB mount, http://cherryamericas.com/wp-content/uploads/2014/12/mx_cat.pdf")
 		(tags "Cherry MX keyswitch 1.00u PCB")
@@
 	(footprint "footprints:SW_Cherry_MX_1.00u_PCB"
 		(layer "F.Cu")
-		(at 227.785 88.439125)
+		(at 218.6 88.439125)
 		(descr "Cherry MX keyswitch, 1.00u, PCB mount, http://cherryamericas.com/wp-content/uploads/2014/12/mx_cat.pdf")
 		(tags "Cherry MX keyswitch 1.00u PCB")
@@
 	(footprint "footprints:SW_Cherry_MX_1.00u_PCB"
 		(layer "F.Cu")
-		(at 116.8 88.439125)
+		(at 123.71 88.439125)
 		(descr "Cherry MX keyswitch, 1.00u, PCB mount, http://cherryamericas.com/wp-content/uploads/2014/12/mx_cat.pdf")
 		(tags "Cherry MX keyswitch 1.00u PCB")
@@
 	(footprint "MountingHole:MountingHole_3.2mm_M3"
 		(layer "F.Cu")
-		(at 66 77)
+		(at 82.67 77)
 		(descr "Mounting Hole 3.2mm, M3, no annular, generated by kicad-footprint-generator mountinghole.py")
 		(tags "mountinghole M3")
@@
 		)
 		(property "Value" "MountingHole_3.2mm_M3"
-			(at 0 4.15 0)
+			(at 0.46 4.15 0)
 			(layer "F.Fab")
 			(effects
@@
 	(footprint "footprints:SW_Cherry_MX_1.00u_PCB"
 		(layer "F.Cu")
-		(at 73.79 88.439125)
+		(at 85.21 88.439125)
 		(descr "Cherry MX keyswitch, 1.00u, PCB mount, http://cherryamericas.com/wp-content/uploads/2014/12/mx_cat.pdf")
 		(tags "Cherry MX keyswitch 1.00u PCB")
@@
 	(footprint "footprints:SW_Cherry_MX_1.00u_PCB"
 		(layer "F.Cu")
-		(at 249.29 88.439125)
+		(at 237.87 88.439125)
 		(descr "Cherry MX keyswitch, 1.00u, PCB mount, http://cherryamericas.com/wp-content/uploads/2014/12/mx_cat.pdf")
 		(tags "Cherry MX keyswitch 1.00u PCB")
@@
 	(footprint "MountingHole:MountingHole_3.2mm_M3"
 		(layer "F.Cu")
-		(at 252 77)
+		(at 235.33 77)
 		(descr "Mounting Hole 3.2mm, M3, no annular, generated by kicad-footprint-generator mountinghole.py")
 		(tags "mountinghole M3")
@@
 		(tags "connector JST XH vertical")
 		(property "Reference" "J101"
-			(at 5 -5.920875 0)
+			(at 4.54 -5.920875 0)
 			(layer "B.SilkS")
 			(effects
@@
 		)
 		(property "Value" "LeftKeyConnector"
-			(at 5 -4.6 0)
+			(at 4.54 -4.6 0)
 			(layer "B.Fab")
 			(effects
@@
 	)
 	(gr_rect
-		(start 60 70)
-		(end 258 104)
+		(start 72.5 70)
+		(end 245.5 104)
+		(radius 2)
 		(stroke
 			(width 0.2)
-			(type default)
+			(type solid)
 		)
 		(fill no)
@@
 	)
 	(gr_text "Designed by github.com/Mircas001\n"
-		(at 230 72 0)
+		(at 176.75 72.25 0)
 		(layer "F.SilkS")
 		(effects
@@
 		)
 	)
+	(gr_text "AnaDash\nInputBoard"
+		(at 165.9 83.6 0)
+		(layer "F.SilkS")
+		(effects
+			(font
+				(size 3 3)
+				(bold yes)
+			)
+			(justify left bottom)
+		)
+	)
 	(gr_text "SW1"
 		(at 102.310625 70.4 90)
@@
 	)
 	(segment
-		(start 121.4 88.439125)
-		(end 138.305 88.439125)
+		(start 118.560875 85.6)
+		(end 140.120875 85.6)
 		(width 0.2)
 		(layer "F.Cu")
@@
 	(segment
 		(start 109.24 76.279125)
-		(end 121.4 88.439125)
+		(end 118.560875 85.6)
+		(width 0.2)
+		(layer "F.Cu")
+		(net "Net-(J101-Pin_2)")
+	)
+	(segment
+		(start 140.120875 85.6)
+		(end 142.96 88.439125)
 		(width 0.2)
 		(layer "F.Cu")
@@
 	)
 	(segment
+		(start 166.25 96.724125)
+		(end 159.84 90.314125)
+		(width 0.2)
+		(layer "F.Cu")
+		(net "GND")
+	)
+	(segment
 		(start 151.75 79.369125)
 		(end 154.84 76.279125)
@@
 	)
 	(segment
-		(start 156.8 90.969125)
-		(end 151.75 96.019125)
+		(start 156.8 90.994125)
+		(end 151.75 96.044125)
 		(width 0.2)
 		(layer "F.Cu")
@@
 	)
 	(segment
-		(start 159.84 84.609125)
-		(end 159.84 76.279125)
+		(start 166.25 91.019125)
+		(end 159.84 84.609125)
 		(width 0.2)
 		(layer "F.Cu")
@@
 	)
 	(segment
-		(start 166.25 91.019125)
-		(end 159.84 84.609125)
+		(start 159.84 84.609125)
+		(end 159.84 76.279125)
 		(width 0.2)
 		(layer "F.Cu")
@@
 	)
 	(segment
-		(start 95.295 85.224125)
+		(start 104.46 76.499125)
 		(end 104.24 76.279125)
 		(width 0.2)
@@
 	)
 	(segment
-		(start 95.295 88.439125)
-		(end 95.295 85.224125)
+		(start 104.46 88.439125)
+		(end 104.46 76.499125)
 		(width 0.2)
 		(layer "F.Cu")
@@
 	)
 	(segment
-		(start 206.28 88.439125)
-		(end 217.54 77.179125)
+		(start 199.37 88.439125)
+		(end 205.38 88.439125)
 		(width 0.2)
 		(layer "F.Cu")
@@
 	)
 	(segment
-		(start 217.54 77.179125)
+		(start 205.38 88.439125)
 		(end 217.54 76.279125)
 		(width 0.2)
@@
 	)
 	(segment
-		(start 184.775 88.439125)
-		(end 202.88 88.439125)
+		(start 204.28 87.039125)
+		(end 215.04 76.279125)
 		(width 0.2)
 		(layer "F.Cu")
@@
 	)
 	(segment
-		(start 202.88 88.439125)
-		(end 215.04 76.279125)
+		(start 180.1 88.439125)
+		(end 181.5 87.039125)
+		(width 0.2)
+		(layer "F.Cu")
+		(net "Net-(J102-Pin_5)")
+	)
+	(segment
+		(start 181.5 87.039125)
+		(end 204.28 87.039125)
 		(width 0.2)
 		(layer "F.Cu")
@@
 	)
 	(segment
-		(start 227.785 88.439125)
-		(end 227.785 84.024125)
+		(start 218.6 88.439125)
+		(end 218.6 77.719125)
 		(width 0.2)
 		(layer "F.Cu")
@@
 	)
 	(segment
-		(start 227.785 84.024125)
+		(start 218.6 77.719125)
 		(end 220.04 76.279125)
 		(width 0.2)
@@
 	)
 	(segment
-		(start 116.8 88.439125)
-		(end 116.8 86.339125)
+		(start 123.71 88.439125)
+		(end 118.9 88.439125)
 		(width 0.2)
 		(layer "F.Cu")
@@
 	)
 	(segment
-		(start 116.8 86.339125)
+		(start 118.9 88.439125)
 		(end 106.74 76.279125)
 		(width 0.2)
@@
 	)
 	(segment
-		(start 73.79 88.439125)
+		(start 85.21 88.439125)
 		(end 89.58 88.439125)
 		(width 0.2)
@@
 	)
 	(segment
-		(start 249.29 88.439125)
-		(end 234.7 88.439125)
+		(start 234.7 88.439125)
+		(end 222.54 76.279125)
 		(width 0.2)
 		(layer "F.Cu")
@@
 	)
 	(segment
-		(start 234.7 88.439125)
-		(end 222.54 76.279125)
+		(start 237.87 88.439125)
+		(end 234.7 88.439125)
 		(width 0.2)
 		(layer "F.Cu")
@@
 		(polygon
 			(pts
-				(xy 258 70) (xy 258 105) (xy 60 105) (xy 60 70)
+				(xy 245.5 70) (xy 245.5 105) (xy 72.5 105) (xy 72.5 70)
 			)
 		)
